File: main_v3.brd (EAGLE design)
At the start: 103.8 x 81.3 mm, 22 parts, among them U1 CD4026BE, U2 CD4026BE

Commit message: load
Parts:
- moved U2 13.5 mm to (78.7, 66.0)
- moved U1 11.7 mm to (20.3, 47.0)
- turned R15 to 0 degrees
Connections:
- net GND: now also SV1.2; no longer SV1.4
- net N$32: now also SV1.4; no longer SV1.2
