File: main_v3.sch (EAGLE design)
At the start: 22 parts, among them U1 CD4026BE, U2 CD4026BE

Commit message: load
Connections:
- net GND: now also SV1.2; no longer SV1.4
- net N$32: now also SV1.4; no longer SV1.2
Changed lines of the file:
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@@
 <net name="GND" class="0">
 <segment>
-<pinref part="SV1" gate="1" pin="4"/>
-<wire x1="104.14" y1="106.68" x2="109.22" y2="114.3" width="0.1524" layer="91"/>
+<pinref part="SV1" gate="1" pin="2"/>
+<wire x1="104.14" y1="106.68" x2="104.14" y2="114.3" width="0.1524" layer="91"/>
 <pinref part="SUPPLY3" gate="GND" pin="GND"/>
 </segment>
@@
 <wire x1="213.36" y1="7.62" x2="210.82" y2="7.62" width="0.1524" layer="91"/>
 <wire x1="210.82" y1="7.62" x2="210.82" y2="-7.62" width="0.1524" layer="91"/>
-<pinref part="SV1" gate="1" pin="2"/>
-<wire x1="104.14" y1="114.3" x2="109.22" y2="111.76" width="0.1524" layer="91"/>
+<pinref part="SV1" gate="1" pin="4"/>
+<wire x1="109.22" y1="114.3" x2="109.22" y2="111.76" width="0.1524" layer="91"/>
 <wire x1="109.22" y1="111.76" x2="149.86" y2="111.76" width="0.1524" layer="91"/>
 <wire x1="210.82" y1="-7.62" x2="149.86" y2="-7.62" width="0.1524" layer="91"/>
