File: main.brd (EAGLE design)
At the start: 103.8 x 81.3 mm, 23 parts, among them U1 CD4026B_N_16, U2 CD4026B_N_16

Commit message: Add v4 mirror drivers
Parts:
- moved R17 42.4 mm to (73.7, 5.08), turned to 90 degrees
- moved R14 29.2 mm to (33.0, 24.1)
- moved R2 29.2 mm to (63.5, 24.1)
- moved R1 29.2 mm to (63.5, 26.7)
- moved R11 29.2 mm to (33.0, 14.0)
- moved R12 29.2 mm to (33.0, 11.4)
- moved R13 29.2 mm to (33.0, 26.7)
- moved R15 29.2 mm to (85.1, 5.08), turned to 270 degrees
- moved R16 29.2 mm to (8.89, 8.89)
- moved R18 29.2 mm to (77.5, 5.08)
- moved R3 29.2 mm to (63.5, 11.4)
- moved R4 29.2 mm to (63.5, 14.0)
- moved U1 29.2 mm to (21.6, 11.4)
- moved LED1 29.2 mm to (41.9, 19.1)
- moved LED2 29.2 mm to (54.6, 19.1)
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Routing:
- net N$9: track 240.1 -> 199.4 mm
- net N$28: track 44.3 -> 48.1 mm
- net N$27: track 109.4 -> 105.8 mm
- net N$26: track 157.8 -> 160.5 mm
- net N$22: track 24.7 -> 22.2 mm
Other:
- board size 103.8 x 81.3 mm -> 88.6 x 33 mm
