File: main_v4.brd (EAGLE design)
At the start: 152.1 x 77.5 mm, 22 parts, among them U1 CD4026B_N_16, U2 CD4026B_N_16

Commit message: last
Parts:
- moved R17 6.35 mm to (52.1, 50.8)
- moved R16 1.80 mm to (5.08, 49.5)
Routing:
- net N$20: track 122.1 -> 108.3 mm
- net N$9: track 200.1 -> 189.1 mm
- net N$17: track 33.1 -> 31.7 mm
- net N$31: track 21.8 -> 20.6 mm
- net N$28: track 11.8 -> 12.7 mm
- net N$33: track 26.1 -> 26.9 mm
Changed lines of the file:
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@@
 <element name="R14" library="resistor" package="R0805" value="220" x="27.94" y="44.45"/>
 <element name="R15" library="resistor" package="R0805" value="10K" x="80.01" y="43.18" rot="R270"/>
-<element name="R16" library="resistor" package="R0805" value="10K" x="6.35" y="50.8"/>
-<element name="R17" library="resistor" package="R0805" value="10K" x="58.42" y="50.8"/>
+<element name="R16" library="resistor" package="R0805" value="10K" x="5.08" y="49.53"/>
+<element name="R17" library="resistor" package="R0805" value="10K" x="52.07" y="50.8"/>
 </elements>
 <signals>
@@
 <wire x1="8.89" y1="46.99" x2="8.89" y2="45.72" width="0.254" layer="1"/>
 <wire x1="10.16" y1="48.26" x2="8.89" y2="46.99" width="0.254" layer="1"/>
-<wire x1="17.78" y1="43.18" x2="20.32" y2="45.72" width="0.4064" layer="1"/>
+<wire x1="17.78" y1="43.18" x2="20.32" y2="45.72" width="0.254" layer="1"/>
 <via x="20.32" y="45.72" extent="1-16" drill="0.9" shape="square"/>
 <wire x1="20.32" y1="45.72" x2="24.13" y2="49.53" width="0.4064" layer="16"/>
 <wire x1="24.13" y1="49.53" x2="67.31" y2="49.53" width="0.4064" layer="16"/>
 <via x="67.31" y="49.53" extent="1-16" drill="0.9" shape="square"/>
-<wire x1="67.31" y1="49.53" x2="68.58" y2="48.26" width="0.4064" layer="1"/>
+<wire x1="67.31" y1="49.53" x2="68.58" y2="48.26" width="0.254" layer="1"/>
 </signal>
 <signal name="N$9">
@@
 <wire x1="76.2" y1="27.94" x2="67.31" y2="27.94" width="0.254" layer="1"/>
 <wire x1="76.2" y1="30.48" x2="76.2" y2="27.94" width="0.254" layer="1"/>
-<wire x1="49.53" y1="50.8" x2="57.57" y2="50.8" width="0.254" layer="1"/>
+<wire x1="49.53" y1="50.8" x2="51.22" y2="50.8" width="0.254" layer="1"/>
 <wire x1="49.53" y1="49.53" x2="49.53" y2="50.8" width="0.254" layer="1"/>
 <wire x1="76.2" y1="45.72" x2="80.01" y2="41.91" width="0.254" layer="1"/>
@@
 <wire x1="80.01" y1="41.91" x2="80.01" y2="34.29" width="0.254" layer="1"/>
 <wire x1="80.01" y1="41.91" x2="80.01" y2="42.33" width="0.254" layer="1"/>
-<wire x1="24.13" y1="52.07" x2="17.78" y2="45.72" width="0.254" layer="1"/>
-<wire x1="39.37" y1="52.07" x2="24.13" y2="52.07" width="0.254" layer="1"/>
-<wire x1="39.37" y1="49.53" x2="39.37" y2="52.07" width="0.254" layer="1"/>
-<wire x1="15.24" y1="50.8" x2="7.62" y2="50.8" width="0.254" layer="1"/>
-<wire x1="15.24" y1="48.26" x2="15.24" y2="50.8" width="0.254" layer="1"/>
-<wire x1="17.78" y1="45.72" x2="15.24" y2="48.26" width="0.254" layer="1"/>
+<wire x1="24.13" y1="50.8" x2="17.78" y2="45.72" width="0.254" layer="1"/>
+<wire x1="39.37" y1="50.8" x2="24.13" y2="50.8" width="0.254" layer="1"/>
+<wire x1="39.37" y1="49.53" x2="39.37" y2="50.8" width="0.254" layer="1"/>
+<wire x1="13.97" y1="49.53" x2="6.35" y2="49.53" width="0.254" layer="1"/>
+<wire x1="17.78" y1="45.72" x2="13.97" y2="49.53" width="0.254" layer="1"/>
 <wire x1="1.27" y1="43.18" x2="3.81" y2="40.64" width="0.254" layer="1"/>
 <wire x1="1.27" y1="44.45" x2="1.27" y2="43.18" width="0.254" layer="1"/>
-<wire x1="7.62" y1="50.8" x2="1.27" y2="44.45" width="0.254" layer="1"/>
-<wire x1="7.62" y1="50.8" x2="7.2" y2="50.8" width="0.254" layer="1"/>
+<wire x1="6.35" y1="49.53" x2="1.27" y2="44.45" width="0.254" layer="1"/>
+<wire x1="6.35" y1="49.53" x2="5.93" y2="49.53" width="0.254" layer="1"/>
 </signal>
 <signal name="N$10">
@@
 <wire x1="0" y1="41.91" x2="0" y2="45.72" width="0.254" layer="1"/>
 <wire x1="3.81" y1="38.1" x2="0" y2="41.91" width="0.254" layer="1"/>
-<wire x1="16.51" y1="49.53" x2="17.78" y2="48.26" width="0.254" layer="1"/>
-<wire x1="16.51" y1="50.8" x2="16.51" y2="49.53" width="0.254" layer="1"/>
-<wire x1="15.24" y1="52.07" x2="16.51" y2="50.8" width="0.254" layer="1"/>
-<wire x1="5.08" y1="52.07" x2="15.24" y2="52.07" width="0.254" layer="1"/>
-<wire x1="5.08" y1="50.8" x2="5.08" y2="52.07" width="0.254" layer="1"/>
-<wire x1="5.08" y1="50.8" x2="5.5" y2="50.8" width="0.254" layer="1"/>
+<wire x1="15.24" y1="50.8" x2="17.78" y2="48.26" width="0.254" layer="1"/>
+<wire x1="5.08" y1="50.8" x2="15.24" y2="50.8" width="0.254" layer="1"/>
+<wire x1="5.08" y1="50.8" x2="4.23" y2="49.53" width="0.254" layer="1"/>
 </signal>
 <signal name="N$18">
@@
 <contactref element="U1" pad="6"/>
 <contactref element="R9" pad="1"/>
-<wire x1="25.4" y1="40.64" x2="27.09" y2="41.91" width="0.254" layer="1"/>
 <wire x1="20.32" y1="35.56" x2="25.4" y2="40.64" width="0.254" layer="1"/>
+<wire x1="25.4" y1="40.64" x2="25.4" y2="41.91" width="0.254" layer="1"/>
+<wire x1="25.4" y1="41.91" x2="27.09" y2="41.91" width="0.254" layer="1"/>
 <wire x1="17.78" y1="35.56" x2="20.32" y2="35.56" width="0.254" layer="1"/>
 </signal>
@@
 <contactref element="U1" pad="12"/>
 <contactref element="R13" pad="1"/>
-<wire x1="19.05" y1="39.37" x2="19.05" y2="40.64" width="0.254" layer="1"/>
-<wire x1="19.05" y1="40.64" x2="26.67" y2="46.99" width="0.254" layer="1"/>
-<wire x1="10.16" y1="39.37" x2="19.05" y2="39.37" width="0.254" layer="1"/>
-<wire x1="10.16" y1="38.1" x2="10.16" y2="39.37" width="0.254" layer="1"/>
-<wire x1="26.67" y1="46.99" x2="27.09" y2="46.99" width="0.254" layer="1"/>
+<wire x1="19.05" y1="41.91" x2="24.13" y2="46.99" width="0.254" layer="1"/>
+<wire x1="24.13" y1="46.99" x2="27.09" y2="46.99" width="0.254" layer="1"/>
+<wire x1="13.97" y1="41.91" x2="19.05" y2="41.91" width="0.254" layer="1"/>
+<wire x1="10.16" y1="38.1" x2="13.97" y2="41.91" width="0.254" layer="1"/>
 </signal>
 <signal name="N$32">
@@
 <contactref element="U1" pad="10"/>
 <contactref element="R14" pad="1"/>
-<wire x1="20.32" y1="36.83" x2="26.67" y2="44.45" width="0.254" layer="1"/>
-<wire x1="8.89" y1="36.83" x2="20.32" y2="36.83" width="0.254" layer="1"/>
+<wire x1="19.05" y1="36.83" x2="22.86" y2="40.64" width="0.254" layer="1"/>
+<wire x1="22.86" y1="40.64" x2="22.86" y2="42.65395" width="0.254" layer="1"/>
+<wire x1="22.86" y1="42.65395" x2="24.65605" y2="44.45" width="0.254" layer="1"/>
+<wire x1="24.65605" y1="44.45" x2="27.09" y2="44.45" width="0.254" layer="1"/>
+<wire x1="8.89" y1="36.83" x2="19.05" y2="36.83" width="0.254" layer="1"/>
 <wire x1="8.89" y1="34.29" x2="8.89" y2="36.83" width="0.254" layer="1"/>
 <wire x1="10.16" y1="33.02" x2="8.89" y2="34.29" width="0.254" layer="1"/>
-<wire x1="26.67" y1="44.45" x2="27.09" y2="44.45" width="0.254" layer="1"/>
 </signal>
 <signal name="N$34">
@@
 <contactref element="R15" pad="1"/>
 <contactref element="U1" pad="5"/>
-<wire x1="17.78" y1="38.1" x2="20.32" y2="39.37" width="0.4064" layer="1"/>
-<via x="20.32" y="39.37" extent="1-16" drill="0.9" shape="square"/>
-<wire x1="20.32" y1="39.37" x2="30.48" y2="48.26" width="0.4064" layer="16"/>
+<wire x1="17.78" y1="38.1" x2="20.32" y2="40.64" width="0.254" layer="1"/>
+<via x="20.32" y="40.64" extent="1-16" drill="0.9" shape="square"/>
+<wire x1="20.32" y1="40.64" x2="30.48" y2="48.26" width="0.4064" layer="16"/>
 <wire x1="30.48" y1="48.26" x2="78.74" y2="48.26" width="0.4064" layer="16"/>
 <via x="78.74" y="48.26" extent="1-16" drill="0.9" shape="square"/>
-<wire x1="78.74" y1="48.26" x2="76.2" y2="48.26" width="0.4064" layer="1"/>
+<wire x1="78.74" y1="48.26" x2="76.2" y2="48.26" width="0.254" layer="1"/>
 <wire x1="78.74" y1="45.72" x2="80.01" y2="44.45" width="0.254" layer="1"/>
 <wire x1="78.74" y1="48.26" x2="78.74" y2="45.72" width="0.254" layer="1"/>
@@
 <wire x1="8.89" y1="40.64" x2="8.89" y2="44.45" width="0.254" layer="1"/>
 <wire x1="8.89" y1="44.45" x2="10.16" y2="45.72" width="0.254" layer="1"/>
-<wire x1="58.42" y1="49.53" x2="59.69" y2="50.8" width="0.254" layer="1"/>
-<wire x1="53.34" y1="49.53" x2="58.42" y2="49.53" width="0.254" layer="1"/>
-<wire x1="53.34" y1="45.72" x2="53.34" y2="49.53" width="0.254" layer="1"/>
+<wire x1="53.34" y1="45.72" x2="53.34" y2="50.8" width="0.254" layer="1"/>
 <wire x1="54.61" y1="44.45" x2="53.34" y2="45.72" width="0.254" layer="1"/>
 <wire x1="55.88" y1="44.45" x2="54.61" y2="44.45" width="0.254" layer="1"/>
@@
 <wire x1="-1.27" y1="40.64" x2="3.81" y2="35.56" width="0.254" layer="1"/>
 <wire x1="-1.27" y1="46.99" x2="-1.27" y2="40.64" width="0.254" layer="1"/>
-<wire x1="5.08" y1="53.34" x2="-1.27" y2="46.99" width="0.254" layer="1"/>
-<wire x1="59.69" y1="53.34" x2="5.08" y2="53.34" width="0.254" layer="1"/>
-<wire x1="59.69" y1="50.8" x2="59.69" y2="53.34" width="0.254" layer="1"/>
-<wire x1="59.69" y1="50.8" x2="59.27" y2="50.8" width="0.254" layer="1"/>
+<wire x1="3.81" y1="52.07" x2="-1.27" y2="46.99" width="0.254" layer="1"/>
+<wire x1="53.34" y1="52.07" x2="3.81" y2="52.07" width="0.254" layer="1"/>
+<wire x1="53.34" y1="50.8" x2="53.34" y2="52.07" width="0.254" layer="1"/>
+<wire x1="53.34" y1="50.8" x2="52.92" y2="50.8" width="0.254" layer="1"/>
 </signal>
 </signals>
-<errors>
-</errors>
 </board>
 </drawing>
